File: KICAD/BTMS.kicad_sch (KiCad schematic)
At the start: 230 parts, among them J1 Batt_Ballance, J10 PWR_SW, J2 USB_C_Receptacle_4085, J3 AUX_Charge, J4 Battery_IO, J5 Power_Out, J6 DSKY, J7 BatteryPTC, J8 Heater, J9 ICSP, Q2 SSM3K341R, Q3 BSS84-7-F, Q4 DMN65D8L, Q5 DMN65D8L, Q6 SSM3K341R, Q7 DMN65D8L, Q8 DMN65D8L, SW1 PTS526, U1 FAN3100TSX, U10 ACS711xLCTR-25AB, U11 ISL95808HRZ, U12 AON7522E, U13 AON7522E, U14 AONR21321, U15 AON7522E, U16 LM62CIM3/NOPB, U17 FAN3100TSX, U18 AP62250Z6, U19 AP62250Z6, U20 dsPIC30F4011-PT, U21 FT230XQ, U22 MIC5504-3.3YM5, U23 DMP2240UDM, U24 DMP2240UDM, U25 DMP2240UDM, U26 DMP2240UDM, U27 AONR21321, U28 FAN3100TSX, U29 ISL95808HRZ, U3 Q294700DSGR, U30 AON7522E, U31 DMP2240UDM, U32 MCP3021, U4 ACS711xLCTR-25AB, U5 IS281-4, U6 SCF4030-12-0X, U7 AP33772, U8 IS281-4, U9 AONR21321

Commit message: Replaced USB-C input diode with P-Channel MOSFET array controlled by dsPIC and USB-PD chip. Added IO expanded chip for dsPIC and USB-C input control interface. Moved some things around on board layout.
Parts:
- removed D1: SBRT15U50SP5-13, Package_TO_SOT_SMD:TO-277B, symbol Device:D_Schottky_AAK
- added C73: 0.1uf, Capacitor_SMD:C_0402_1005Metric, symbol Device:C
- added D1: BAV23CLT1G, Package_TO_SOT_SMD:SOT-23, symbol Diode:BAV70
- added D7: D_Schottky40V, Diode_SMD:D_0603_1608Metric, symbol Device:D
- added Q1: DMN65D8L, Package_TO_SOT_SMD:SOT-23, symbol Device:Q_NMOS_GSD
- added R10: 5K, Resistor_SMD:R_0603_1608Metric, symbol Device:R
- added R16, R8: 1K, Resistor_SMD:R_0603_1608Metric, symbol Device:R
- added U2, U33: AONR21321, Package_DFN_QFN:DFN-8-1EP_3x3mm_P0.65mm_EP1.7x2.05mm, symbol New_Library:AONR21321
- added U34: PCA9570GMH, XQFN8_SOT902-2_NXP, symbol 2024-07-18_22-04-03:PCA9570GMH
Connections:
- net +3V3: now also C73.1, U34.8 (VDD)
- net GND: now also C73.2, Q1.2 (S), R8.2, U34.4 (VSS)
- net at C63.1, R17.2, U7.1 (ISENP): now also R16.2, U33.5 (D), U33.6 (D), U33.7 (D), U33.8 (D), U33.9 (D)
- net at F1.2: now also D7.2 (A), U2.5 (D), U2.6 (D), U2.7 (D), U2.8 (D), U2.9 (D)
- net PD_Enable: now reaches U7.23 (PWR_EN)
- net PD_Enable: now also D1.2 (A)
- net PGMC renamed ISDA
- net ISDA: now also U34.7 (SDA)
- net PGMD renamed ISCL
- net ISCL: now also U34.6 (SCL)
- new net: R10.1, U2.1 (S), U2.2 (S), U2.3 (S), U33.1 (S), U33.2 (S), U33.3 (S)
- new net: Q1.3 (D), R10.2, U2.4 (G), U33.4 (G)
- new net: D7.1 (K), R16.1
- new net: D1.3 (K), Q1.1 (G), R8.1
- new net USB_Enable: D1.1 (A), U34.1 (P0)
Other:
- note added: "IO Expansion"
- moved on the sheet: C11, C19, C21, C32, C37, C38, C44, C45, C49, C50, C52, C53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
